File: powerboard_v2.kicad_pcb (KiCad board)
At the start: 2 copper layers, 70 x 70 mm, 34 parts, among them J1 Conn_01x02_Pin, J2 Conn_01x02_Pin, J3 Conn_01x02_Pin, J4 Conn_01x02_Pin, J5 Conn_01x02_Pin, K3 Relay_SPDT, U2 BD99010EFV-ME2, U5 TLP785

Commit message: 変更していたらしい
Parts:
- moved G*** 24.9 mm to (83.2, 108.2)
Routing:
- net GND2: track 24.0 -> 48.4 mm
- net Net-(L1-Pad1): track 15.5 -> 31.2 mm
- net xt60_out: track 30.9 -> 34.3 mm
- net GND: track 13.2 -> 16.5 mm, vias 0 -> 56
- net cap out: track 11.5 -> 12.7 mm
Other:
- board text added: "+ -"
